Commit message: updates

File: ros2ws/src/ros2_gopigo3_node/urdf/humbledave2.urdf (robot description, URDF)
Before this commit: robot humbledave2_v25_04_06, 10 links, 9 joints
Links:
- removed link base_footprint
- removed link base_scan
- removed link camera_link
- removed link camera_rgb_frame
- removed link gopi5go_dave_link
- removed link wheel_left_link
- removed link wheel_right_link
- added link dave_link; visual cylinder length=0.008 radius=0.015; visual cylinder length=0.008 radius=0.015
- added link laser_frame; visual cylinder length=0.020 radius=0.0325
- added link left_wheel; visual cylinder length=0.025 radius=0.03385
- added link oak_d_w_frame; visual box size=0.022 0.097 0.030
- added link right_wheel; visual cylinder length=0.025 radius=0.033385
- link base_link: geometry visual box size=0.025 0.055 0.002; visual box size=0.128 0.104 0.004
Joints:
- removed joint base_joint
- removed joint camera_joint
- removed joint camera_rgb_joint
- removed joint wheel_left_joint
- removed joint wheel_right_joint
- added joint joint_left_wheel: type continuous, parent base_link, child left_wheel, origin xyz=0 0.058 0.033385 rpy=0 0 0, axis 0 1 0
- added joint joint_oak_d_w: type fixed, parent base_link, child oak_d_w_frame, origin xyz=0.08 0 0.162 rpy=0 0 0
- added joint joint_right_wheel: type continuous, parent base_link, child right_wheel, origin xyz=0 -0.058 0.033385 rpy=0 0 0, axis 0 1 0
- joint joint_dave: child gopi5go_dave_link -> dave_link; origin xyz=-0.04 0 0.2045615 rpy=0 0 0 -> xyz=-0.04 0 0.250 rpy=0 0 0
- joint joint_dave_eyes: origin xyz=-0.04 0 0.2045615 rpy=0 0 0 -> xyz=-0.04 0 0.250 rpy=0 0 0
- joint joint_imu: origin xyz=0.070 0.035 0.0535615 rpy=0 0 0 -> xyz=0.070 0.035 0.104 rpy=0 0 0
- joint joint_ydlidar: child base_scan -> laser_frame; origin xyz=-0.014 0 0.1545615 rpy=0 0 0 -> xyz=-0.014 0 0.200 rpy=0 0 0
